File: Hardware/PCB_Design/PCB_Design.kicad_pcb (KiCad board)
At the start: 2 copper layers, 146.1 x 78.7 mm, 16 parts, among them J1 Conn_01x02_Male, J2 Conn_01x03_Male, J3 Conn_01x03_Male, J4 Conn_01x02_Male, U1 LM7805_TO220, U2 ESP32-CAM, U3 L298HN

Commit message: renamed project
Parts:
- added BT2: Battery_Cell, Battery:BatteryHolder_MPD_BH-18650-PC2, F.Cu at (57.8, 78.7)
- added C1: C_Polarized, Capacitor_SMD:CP_Elec_3x5.3, F.Cu at (157.9, 100.3)
- added C2: C_Polarized, Capacitor_SMD:CP_Elec_3x5.3, F.Cu at (158.0, 120.7)
- added J5: Conn_01x02_Male, Connector_PinHeader_1.00mm:PinHeader_1x02_P1.00mm_Vertical, F.Cu at (111.1, 99.1)
- added J6: Conn_01x02_Male, Connector_PinHeader_1.00mm:PinHeader_1x02_P1.00mm_Vertical, F.Cu at (170.8, 99.3)
- moved J3 82.0 mm to (169.5, 116.8)
- moved J2 26.2 mm to (169.5, 111.8)
- moved J4 23.3 mm to (169.5, 122.2)
- moved U1 22.7 mm to (164.5, 113.8)
- moved D1 21.9 mm to (130.2, 99.1), turned to -90 degrees
- moved D5 21.9 mm to (145.4, 99.1), turned to -90 degrees
- moved D2 21.8 mm to (130.2, 113.3), turned to -90 degrees
- moved D3 21.8 mm to (137.7, 99.1), turned to -90 degrees
- moved D6 21.7 mm to (145.3, 113.3), turned to -90 degrees
- moved D4 21.7 mm to (137.7, 113.3), turned to -90 degrees
- moved D7 21.5 mm to (151.4, 99.1), turned to -90 degrees
- moved D8 21.5 mm to (151.4, 113.3), turned to -90 degrees
- moved U3 21.3 mm to (120.8, 111.9)
- moved J1 9.69 mm to (51.4, 68.6), turned to 180 degrees
- moved BT1 8.25 mm to (57.3, 57.1)
Connections:
- J1 pad 1: Net-(BT1-Pad2) -> Net-(J1-Pad1)
- J4 pad 1: Net-(J4-Pad1) -> Net-(U1-Pad1)
- U1 pad 1: unconnected-(U1-Pad1) -> Net-(U1-Pad1)
- U1 pad 3: Net-(J4-Pad1) -> /VDD
- U3 pad 9: Net-(J4-Pad1) -> /VDD
Routing:
- net GND: track 0.00 -> 79.5 mm
- net Net-(D1-Pad1): track 0.00 -> 46.1 mm
- net /OUT4: track 0.00 -> 38.8 mm
- net /OUT3: track 0.00 -> 28.9 mm
- net /OUT2: track 0.00 -> 28.2 mm
- net /OUT1: track 0.00 -> 24.9 mm
- net /VDD: track 0.00 -> 21.2 mm
- net Net-(U1-Pad1): track 0.00 -> 12.0 mm
Other:
- board size 146.1 x 78.7 mm -> 154.3 x 81.3 mm
