File: Hardware/PCB_Design/PCB_Design.kicad_sch (KiCad schematic)
At the start: 21 parts, among them J1 Conn_01x02_Male, J2 Conn_01x03_Male, J3 Conn_01x03_Male, J4 Conn_01x02_Male, J5 Conn_01x02_Male, J6 Conn_01x02_Male, U1 LM7805_TO220, U2 ESP32-CAM, U3 L298HN

Commit message: renamed project
Parts:
- removed C1, C2: 220u, Capacitor_SMD:CP_Elec_3x5.3, symbol Device:C
- added C1, C2: C_Polarized, Capacitor_SMD:CP_Elec_3x5.3, symbol Device:C_Polarized
Connections:
- net GND: now also C1.2, C2.2
- net VDD: now also C1.1
- net at D1.1 (K), D3.1 (K), D5.1 (K)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: now also C2.1
Changed lines of the file:
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@@
   (junction (at 205.74 102.235) (diameter 0) (color 0 0 0 0)
   )
+  (junction (at 135.255 69.215) (diameter 0) (color 0 0 0 0)
+  )
   (junction (at 191.135 116.205) (diameter 0) (color 0 0 0 0)
   )
@@
   )
   (junction (at 124.46 78.105) (diameter 0) (color 0 0 0 0)
-  )
-  (junction (at 135.255 69.215) (diameter 0) (color 0 0 0 0)
   )
   (no_connect (at 66.04 30.48))
@@
   (no_connect (at 66.04 53.34))
   (no_connect (at 66.04 49.53))
+  (wire (pts (xy 135.255 69.215) (xy 158.115 69.215))
+    (stroke (width 0) (type default) (color 0 0 0 0))
+  )
   (wire (pts (xy 67.31 97.79) (xy 67.31 105.41))
     (stroke (width 0) (type default) (color 0 0 0 0))
@@
     (stroke (width 0) (type default) (color 0 0 0 0))
   )
+  (wire (pts (xy 124.46 78.105) (xy 124.46 80.645))
+    (stroke (width 0) (type default) (color 0 0 0 0))
+  )
+  (wire (pts (xy 173.355 118.745) (xy 201.295 118.745))
+    (stroke (width 0) (type default) (color 0 0 0 0))
+  )
+  (wire (pts (xy 173.355 116.205) (xy 191.135 116.205))
+    (stroke (width 0) (type default) (color 0 0 0 0))
+  )
+  (wire (pts (xy 135.255 76.835) (xy 135.255 78.105))
+    (stroke (width 0) (type default) (color 0 0 0 0))
+  )
+  (wire (pts (xy 150.495 146.685) (xy 153.035 146.685))
+    (stroke (width 0) (type default) (color 0 0 0 0))
+  )
+  (wire (pts (xy 160.655 103.505) (xy 160.655 86.995))
+    (stroke (width 0) (type default) (color 0 0 0 0))
+  )
+  (wire (pts (xy 191.135 140.335) (xy 201.295 140.335))
+    (stroke (width 0) (type default) (color 0 0 0 0))
+  )
+  (wire (pts (xy 205.74 102.235) (xy 210.185 102.235))
+    (stroke (width 0) (type default) (color 0 0 0 0))
+  )
+  (wire (pts (xy 67.31 105.41) (xy 48.895 105.41))
+    (stroke (width 0) (type default) (color 0 0 0 0))
+  )
+  (wire (pts (xy 124.46 76.835) (xy 124.46 78.105))
+    (stroke (width 0) (type default) (color 0 0 0 0))
+  )
   (wire (pts (xy 132.08 69.215) (xy 135.255 69.215))
-    (stroke (width 0) (type default) (color 0 0 0 0))
-  )
-  (wire (pts (xy 124.46 78.105) (xy 124.46 80.645))
-    (stroke (width 0) (type default) (color 0 0 0 0))
-  )
-  (wire (pts (xy 173.355 118.745) (xy 201.295 118.745))
-    (stroke (width 0) (type default) (color 0 0 0 0))
-  )
-  (wire (pts (xy 173.355 116.205) (xy 191.135 116.205))
-    (stroke (width 0) (type default) (color 0 0 0 0))
-  )
-  (wire (pts (xy 135.255 76.835) (xy 135.255 78.105))
-    (stroke (width 0) (type default) (color 0 0 0 0))
-  )
-  (wire (pts (xy 150.495 146.685) (xy 153.035 146.685))
-    (stroke (width 0) (type default) (color 0 0 0 0))
-  )
-  (wire (pts (xy 160.655 103.505) (xy 160.655 86.995))
-    (stroke (width 0) (type default) (color 0 0 0 0))
-  )
-  (wire (pts (xy 191.135 140.335) (xy 201.295 140.335))
-    (stroke (width 0) (type default) (color 0 0 0 0))
-  )
-  (wire (pts (xy 205.74 102.235) (xy 210.185 102.235))
-    (stroke (width 0) (type default) (color 0 0 0 0))
-  )
-  (wire (pts (xy 67.31 105.41) (xy 48.895 105.41))
-    (stroke (width 0) (type default) (color 0 0 0 0))
-  )
-  (wire (pts (xy 124.46 76.835) (xy 124.46 78.105))
-    (stroke (width 0) (type default) (color 0 0 0 0))
-  )
-  (wire (pts (xy 135.255 69.215) (xy 158.115 69.215))
     (stroke (width 0) (type default) (color 0 0 0 0))
   )
@@
   )
   (label "OUT1" (at 173.355 116.205 0)
+    (effects (font (size 1.27 1.27)) (justify left bottom))
+  )
+  (label "Vout" (at 133.35 69.215 0)
     (effects (font (size 1.27 1.27)) (justify left bottom))
   )
@@
     (pin "2")
   )
-  (symbol (lib_id "Device:C") (at 229.87 106.045 0) (unit 1)
-    (in_bom yes) (on_board yes) (fields_autoplaced)
-    (property "Reference" "C2" (id 0) (at 233.68 104.7749 0)
-      (effects (font (size 1.27 1.27)) (justify left))
-    )
-    (property "Value" "220u" (id 1) (at 233.68 107.3149 0)
-      (effects (font (size 1.27 1.27)) (justify left))
-    )
-    (property "Footprint" "Capacitor_SMD:CP_Elec_3x5.3" (id 2) (at 230.8352 109.855 0)
-      (effects (font (size 1.27 1.27)) hide)
-    )
-    (property "Datasheet" "~" (id 3) (at 229.87 106.045 0)
+  (symbol (lib_id "Device:C_Polarized") (at 135.255 73.025 0) (unit 1)
+    (in_bom yes) (on_board yes) (fields_autoplaced)
+    (property "Reference" "C1" (id 0) (at 138.43 70.8659 0)
+      (effects (font (size 1.27 1.27)) (justify left))
+    )
+    (property "Value" "C_Polarized" (id 1) (at 138.43 73.4059 0)
+      (effects (font (size 1.27 1.27)) (justify left))
+    )
+    (property "Footprint" "Capacitor_SMD:CP_Elec_3x5.3" (id 2) (at 136.2202 76.835 0)
+      (effects (font (size 1.27 1.27)) hide)
+    )
+    (property "Datasheet" "~" (id 3) (at 135.255 73.025 0)
       (effects (font (size 1.27 1.27)) hide)
     )
@@
     (pin "2")
   )
-  (symbol (lib_id "Device:C") (at 135.255 73.025 0) (unit 1)
-    (in_bom yes) (on_board yes) (fields_autoplaced)
-    (property "Reference" "C1" (id 0) (at 139.065 71.7549 0)
-      (effects (font (size 1.27 1.27)) (justify left))
-    )
-    (property "Value" "220u" (id 1) (at 139.065 74.2949 0)
-      (effects (font (size 1.27 1.27)) (justify left))
-    )
-    (property "Footprint" "Capacitor_SMD:CP_Elec_3x5.3" (id 2) (at 136.2202 76.835 0)
-      (effects (font (size 1.27 1.27)) hide)
-    )
-    (property "Datasheet" "~" (id 3) (at 135.255 73.025 0)
+  (symbol (lib_id "Device:C_Polarized") (at 229.87 106.045 0) (unit 1)
+    (in_bom yes) (on_board yes) (fields_autoplaced)
+    (property "Reference" "C2" (id 0) (at 233.045 103.8859 0)
+      (effects (font (size 1.27 1.27)) (justify left))
+    )
+    (property "Value" "C_Polarized" (id 1) (at 233.045 106.4259 0)
+      (effects (font (size 1.27 1.27)) (justify left))
+    )
+    (property "Footprint" "Capacitor_SMD:CP_Elec_3x5.3" (id 2) (at 230.8352 109.855 0)
+      (effects (font (size 1.27 1.27)) hide)
+    )
+    (property "Datasheet" "~" (id 3) (at 229.87 106.045 0)
       (effects (font (size 1.27 1.27)) hide)
     )
@@
       (reference "BT2") (unit 1) (value "Battery_Cell") (footprint "Battery:BatteryHolder_MPD_BH-18650-PC2")
     )
-    (path "/920e09bb-af07-4798-931b-978c8b013fd3"
-      (reference "C1") (unit 1) (value "220u") (footprint "Capacitor_SMD:CP_Elec_3x5.3")
-    )
-    (path "/71aa8ceb-7f8f-448f-a293-7de428ab4249"
-      (reference "C2") (unit 1) (value "220u") (footprint "Capacitor_SMD:CP_Elec_3x5.3")
+    (path "/71705b42-9471-46d0-90dd-3ba2ae2bcf43"
+      (reference "C1") (unit 1) (value "C_Polarized") (footprint "Capacitor_SMD:CP_Elec_3x5.3")
+    )
+    (path "/89105d90-8ba4-4338-b37e-2a92aca4d814"
+      (reference "C2") (unit 1) (value "C_Polarized") (footprint "Capacitor_SMD:CP_Elec_3x5.3")
     )
     (path "/1c5e17be-93f2-4f06-975a-3e2b5cd83996"
